Commit message: tbot model SDF + URDF + kinect

File: tbot_sim/urdf/tbot.urdf (robot description, URDF)
Before this commit: robot tbot, 12 links, 11 joints
Links:
- removed link wheel_left_link
- removed link wheel_right_link
- added link left_wheel, mass 0.010000; collision cylinder length=0.023000 radius=0.033000; visual mesh filename=package://tbot_sim/models/kobuki/meshes/wheel.dae
- added link right_wheel, mass 0.010000; collision cylinder length=0.023000 radius=0.033000; visual mesh filename=package://tbot_sim/models/kobuki/meshes/wheel.dae
- link base_link: geometry collision cylinder length=0.10938 radius=0.178; visual mesh filename=package://tbot_sim/models/kobuki/meshes/main_body.dae
- link laser_link: geometry collision cylinder length=0.10938 radius=0.178; visual mesh filename=package://tbot_sim/models/hokuyo/meshes/hokuyo.dae
Joints:
- removed joint wheel_left_joint
- removed joint wheel_right_joint
- added joint left_wheel_joint: type fixed, parent base_link, child left_wheel, origin xyz=0 0.115 -0.028 rpy=0 0 0, axis 0 1 0, limit lower=0 upper=0 effort=0 velocity=0
- added joint right_wheel_joint: type fixed, parent base_link, child right_wheel, origin xyz=0 -0.115 -0.028 rpy=0 0 0, axis 0 1 0, limit lower=0 upper=0 effort=0 velocity=0
- joint base_joint: origin xyz=0 0 0.06 rpy=0 0 0 -> xyz=0 0 0.062 rpy=0 0 0
- joint kinect_joint: origin xyz=-0.115 0    0.25 rpy=0 0 0 -> xyz=-0.05 0 0.3 rpy=0 0 0

Commit message: full launch tbot

File: tbot_sim/urdf/tbot.urdf (robot description, URDF)
Before this commit: robot tbot, 12 links, 11 joints
Links:
- removed link kinect_link
- added link camera_link, mass 0.1; collision box size=0.073000 0.276000 0.072000; visual mesh filename=package://tbot_sim/models/kinect/meshes/kinect.dae scale=1.0 1.0 1.0
Joints:
- joint kinect_joint: child kinect_link -> camera_link
